Commit message: Add missing kinect model and fix dependencies

File: urdf/kinect_floating.urdf.xacro (robot description, xacro)
@@ -19,7 +19,7 @@
       <link name="camera_link">
       <visual>
-       <origin xyz="0 0 0" rpy="0 0 ${M_PI/2}"/>
+       <origin xyz="0 0 0" rpy="0 0 0"/>
         <geometry>
-         <mesh filename="package://turtlebot_description/meshes/sensors/kinect.dae"/>
+         <mesh filename="package://costar_objects/sdf/kinect/kinect.dae"/>
         </geometry>
       </visual>
