Commit message: changing the size of the blocks again

File: urdf/block/blue.urdf (robot description, URDF)
Before this commit: robot urdf_robot, 1 links, 0 joints
Links:
- link base_link: geometry collision box size=0.035 0.035 0.035; visual box size=0.035 0.035 0.035

File: urdf/block/green.urdf (robot description, URDF)
Before this commit: robot urdf_robot, 1 links, 0 joints
Links:
- link base_link: geometry collision box size=0.035 0.035 0.035; visual box size=0.035 0.035 0.035

File: urdf/block/red.urdf (robot description, URDF)
Before this commit: robot urdf_robot, 1 links, 0 joints
Links:
- link base_link: geometry collision box size=0.035 0.035 0.035; visual box size=0.035 0.035 0.035

File: urdf/block/yellow.urdf (robot description, URDF)
Before this commit: robot urdf_robot, 1 links, 0 joints
Links:
- link base_link: geometry collision box size=0.035 0.035 0.035; visual box size=0.035 0.035 0.035
